Commit message: upload stereo camera

File: src/jackal_description/urdf/accessories.urdf.xacro (robot description, xacro)
@@ -305,11 +305,11 @@
   <!-- If enabled, generates a pair of flea3 cameras for stereo vision with a tilt of 30 degrees. -->
   <!-- Disabled temporarily due to metapackage issue. -->
-  <xacro:if value="$(optenv JACKAL_STEREO_FLEA3 0)">
-    <xacro:property name="tilt" value="$(optenv JACKAL_FLEA3_TILT 0.5236)"/>
+  <xacro:if value="$(optenv JACKAL_STEREO_FLEA3 1)">
+    <xacro:property name="tilt" value="$(optenv JACKAL_FLEA3_TILT 0)"/>
     <xacro:property name="mount" value="$(optenv JACKAL_FLEA3_MOUNT front)"/>
     <xacro:property name="prefix" value="$(optenv JACKAL_FLEA3_PREFIX ${mount})"/>
     <xacro:property name="parent" value="$(optenv JACKAL_FLEA3_PARENT ${mount}_mount)"/>
-    <xacro:property name="left_name" value="$(optenv JACKAL_FLEA3_LEFT_NAME front/left)"/>
-    <xacro:property name="right_name" value="$(optenv JACKAL_FLEA3_RIGHT_NAME front/right)"/>
+    <xacro:property name="left_name" value="$(optenv JACKAL_FLEA3_LEFT_NAME stereo/left)"/>
+    <xacro:property name="right_name" value="$(optenv JACKAL_FLEA3_RIGHT_NAME stereo/right)"/>
     <xacro:property name="separation" value="$(optenv JACKAL_STEREO_SEPERATION 0.16)"/>
     <xacro:stereo_camera_mount prefix="${prefix}" tilt="${tilt}"/>
